File: hardware/PCB_TopSurface/pfm2_topSurface.kicad_pcb (KiCad board)
At the start: 2 copper layers, 156 x 97.5 mm, 6 parts

Commit message: Fix non-pfm2 sysex problem
Other:
- board text added: "VOL"
- board text added: "preenfm2 - surface control PCB - v1.1"
- board text removed: "preenfm2 - surface control PCB - v1.0"
